File: PCB/BlueSof.sch (KiCad schematic (older format))
At the start: 66 parts, among them SW1 SW_PUSH, SW10 SW_PUSH, SW11 SW_PUSH, SW12 SW_PUSH, SW13 SW_PUSH, SW14 SW_PUSH, SW15 SW_PUSH, SW16 SW_PUSH, SW17 SW_PUSH, SW18 SW_PUSH, SW19 SW_PUSH, SW2 SW_PUSH, SW20 SW_PUSH, SW21 SW_PUSH, SW22 SW_PUSH, SW23 SW_PUSH, SW24 SW_PUSH, SW25 Rotary_Encoder_Switch, SW26 SW_PUSH, SW27 SW_PUSH, SW28 SW_PUSH, SW29 SW_PUSH, SW3 SW_PUSH, SW30 SW_PUSH, SW4 SW_PUSH, SW5 SW_PUSH, SW6 SW_PUSH, SW7 SW_PUSH, SW8 SW_PUSH, SW9 SW_PUSH

Commit message: initial layout
Parts:
- removed TH1, TH3, TH4, TH5, TH6, TH7: HOLE, MountingHole:MountingHole_4mm, symbol SofleKeyboard-rescue:HOLE-Lily58-cache-Lily58_Pro-rescue
- added C1, C2: 4.7uF, Capacitor_SMD:C_0603_1608Metric_Pad1.08x0.95mm_HandSolder, symbol Device:C_Small
- added C3, C4: 22pF, Capacitor_SMD:C_0603_1608Metric_Pad1.08x0.95mm_HandSolder, symbol Device:C_Small
- added C5: 10uF, Capacitor_SMD:C_0603_1608Metric_Pad1.08x0.95mm_HandSolder, symbol Device:C_Small
- added D31, D32: LED, LED_SMD:LED_0603_1608Metric_Pad1.05x0.95mm_HandSolder, symbol Device:LED
- added D33: 1N5819, Diode_SMD:D_SOD-323_HandSoldering, symbol Diode:1N5819
- added J1: USB_C_Receptacle_USB2.0, Connector_USB:USB_C_Receptacle_HRO_TYPE-C-31-M-12, symbol Connector:USB_C_Receptacle_USB2.0
- added J2, J4: Conn_01x01_Female, Connector_PinHeader_2.54mm:PinHeader_1x01_P2.54mm_Vertical, symbol Connector:Conn_01x01_Female
- added J3: Conn_01x04_Female, Connector_PinHeader_2.54mm:PinHeader_1x04_P2.54mm_Vertical, symbol Connector:Conn_01x04_Female
- added Q2: A03407, Package_TO_SOT_SMD:SOT-23, symbol Device:Q_PMOS_GSD
- added R1, R2, R6: 10k, Resistor_SMD:R_0603_1608Metric_Pad0.98x0.95mm_HandSolder, symbol Device:R_Small
- added R4: 820k, Resistor_SMD:R_0603_1608Metric_Pad0.98x0.95mm_HandSolder, symbol Device:R_Small
- added R5: 2M, Resistor_SMD:R_0603_1608Metric_Pad0.98x0.95mm_HandSolder, symbol Device:R_Small
- added R7, R8: 5.1k, Resistor_SMD:R_0603_1608Metric_Pad0.98x0.95mm_HandSolder, symbol Device:R_Small
- added R9: 100k, Resistor_SMD:R_0603_1608Metric_Pad0.98x0.95mm_HandSolder, symbol Device:R_Small
- added SW31: SW_Push, Button_Switch_SMD:SW_SPST_B3U-1000P, symbol Switch:SW_Push
- added U1: LN2054Y42AMR, Package_TO_SOT_SMD:SOT-23-5, symbol ELLOW:LN2054Y42AMR
- added U2: E73-2G4M08S1C, BlueSof:E73-2G4M08S1C-52840, symbol ELLOW:E73-2G4M08S1C
- added U3: AP2112K-3.3, Package_TO_SOT_SMD:SOT-23-5, symbol Regulator_Linear:AP2112K-3.3
- added Y1: 32.768kHz, Crystal:Crystal_SMD_MicroCrystal_CM9V-T1A-2Pin_1.6x1.0mm_HandSoldering, symbol Device:Crystal
- D30: footprint BlueSof:KailhLowProfile -> BlueSof:Diode_SOD123
- SW26: footprint BlueSof:KailhLowProfile -> BlueSof:KailhLowProfile_1.5U
Connections:
- net labels added: BATTERY_MEASURE, DATA+, DATA-, DCCH, P0.02, PROG, RESET, SWC, SWD, VBAT, VBUS, VDD_H
- net labels removed: SW25B, VCC
- wire segments 60 -> 153
- no-connect marks 0 -> 2
Other:
- note added: "BLE Module"
- note added: "Battery Connection"
- note added: "Battery Measure"
- note added: "Debug Header"
- note added: "LiPo Charger"
- note added: "Power & Filtering"
- note added: "Reset"
- note added: "Switch Matrix"
- note added: "USB"
- moved on the sheet: D1, D10, D11, D12, D13, D14, D15, D16, D17, D18, D19, D2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

Commit message: EOD, layout on side 2 done, not routed
Parts:
- added C10: 10uF, Capacitor_SMD:C_0603_1608Metric_Pad1.08x0.95mm_HandSolder, symbol Device:C_Small
- added C6, C7: 22pF, Capacitor_SMD:C_0603_1608Metric_Pad1.08x0.95mm_HandSolder, symbol Device:C_Small
- added C8, C9: 4.7uF, Capacitor_SMD:C_0603_1608Metric_Pad1.08x0.95mm_HandSolder, symbol Device:C_Small
- added D34, D36: LED, LED_SMD:LED_0603_1608Metric_Pad1.05x0.95mm_HandSolder, symbol Device:LED
- added D35: 1N5819, Diode_SMD:D_SOD-323_HandSoldering, symbol Diode:1N5819
- added J5: USB_C_Receptacle_USB2.0, Connector_USB:USB_C_Receptacle_HRO_TYPE-C-31-M-12, symbol Connector:USB_C_Receptacle_USB2.0
- added Q1: A03407, Package_TO_SOT_SMD:SOT-23, symbol Device:Q_PMOS_GSD
- added R10: 2M, Resistor_SMD:R_0603_1608Metric_Pad0.98x0.95mm_HandSolder, symbol Device:R_Small
- added R11, R15, R16: 10k, Resistor_SMD:R_0603_1608Metric_Pad0.98x0.95mm_HandSolder, symbol Device:R_Small
- added R12, R13: 5.1k, Resistor_SMD:R_0603_1608Metric_Pad0.98x0.95mm_HandSolder, symbol Device:R_Small
- added R14: 100k, Resistor_SMD:R_0603_1608Metric_Pad0.98x0.95mm_HandSolder, symbol Device:R_Small
- added R3: 820k, Resistor_SMD:R_0603_1608Metric_Pad0.98x0.95mm_HandSolder, symbol Device:R_Small
- added SW32: SW_Push, Button_Switch_SMD:SW_SPST_B3U-1000P, symbol Switch:SW_Push
- added U4: E73-2G4M08S1C, BlueSof:E73-2G4M08S1C-52840, symbol ELLOW:E73-2G4M08S1C
- added U5: LN2054Y42AMR, Package_TO_SOT_SMD:SOT-23-5, symbol ELLOW:LN2054Y42AMR
- added U6: AP2112K-3.3, Package_TO_SOT_SMD:SOT-23-5, symbol Regulator_Linear:AP2112K-3.3
- added Y2: 32.768kHz, Crystal:Crystal_SMD_MicroCrystal_CM9V-T1A-2Pin_1.6x1.0mm_HandSoldering, symbol Device:Crystal
Connections:
- net labels added: BATTERY_MEASURE2, DCCH2, P0.05, P0.05_2, P0.18, RESET2, VBUS2, VDD_H2
- net labels removed: P0.02, PROG
- wire segments 153 -> 243
- no-connect marks 2 -> 4
Other:
- moved on the sheet: C1, D1, D10, D11, D12, D13, D14, D15, D16, D17, D18, D19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

Commit message: making progress on autoroute cleanup
Changed lines of the file:
@@
 RESET
 Text GLabel 2100 5000 1    50   Input ~ 0
-P0.05_2
+P0.05
 $EndSCHEMATC

Commit message: ordered first boards
Parts:
- R1, R11, R15, R6: value 10k -> 1k
- U4: LCSC Part Number (none) -> BlueSofR1
Connections:
- net labels removed: P0.18
- wire segments 243 -> 241
Other:
- note added: "Back Side"
- note added: "Front Side"
- moved on the sheet: C1, C10, C2, C3, C4, C5, C6, C7, C8, C9, D1, D10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
