File: PCB/BlueSof.kicad_pcb (KiCad board)
At the start: 2 copper layers, 134.3 x 100.2 mm, 174 parts, among them J1 USB_C_Receptacle_USB2.0, J10 Conn_01x01_Female, J2 Conn_01x01_Female, J3 Conn_01x04_Female, J4 Conn_01x01_Female, J5 Conn_01x04_Female, J6 Conn_01x04_Female, J7 USB_C_Receptacle_USB2.0, J8 Conn_01x01_Female, J9 Conn_01x04_Female, Q1 A03407, Q2 A03407, SW1 SW_PUSH, SW10 SW_PUSH, SW11 SW_PUSH, SW12 SW_PUSH, SW13 SW_PUSH, SW14 SW_PUSH, SW15 SW_PUSH, SW16 SW_PUSH, SW17 SW_PUSH, SW18 SW_PUSH, SW19 SW_PUSH, SW2 SW_PUSH, SW20 SW_PUSH, SW21 SW_PUSH, SW22 SW_PUSH, SW23 SW_PUSH, SW24 SW_PUSH, SW25 Rotary_Encoder_Switch, SW26 SW_PUSH, SW27 SW_PUSH, SW28 SW_PUSH, SW29 Rotary_Encoder_Switch, SW3 SW_PUSH, SW30 SW_PUSH, SW31 SW_Push, SW32 SW_PUSH, SW33 SW_PUSH, SW34 SW_PUSH, SW35 SW_PUSH, SW36 SW_PUSH, SW37 SW_PUSH, SW38 SW_PUSH, SW39 SW_PUSH, SW4 SW_PUSH, SW40 SW_PUSH, SW41 SW_PUSH, SW42 SW_PUSH, SW43 SW_PUSH, SW44 SW_PUSH, SW45 SW_Push, SW46 SW_PUSH, SW47 SW_PUSH, SW48 SW_PUSH, SW49 SW_PUSH, SW5 SW_PUSH, SW50 SW_PUSH, SW51 SW_PUSH, SW52 SW_PUSH, SW53 SW_PUSH, SW54 SW_PUSH, SW55 SW_SPDT, SW56 SW_PUSH, SW57 SW_PUSH, SW58 SW_PUSH, SW59 SW_SPDT, SW6 SW_PUSH, SW60 SW_PUSH, SW7 SW_PUSH, SW8 SW_PUSH, SW9 SW_PUSH, U1 LN2054Y42AMR, U2 E73-2G4M08S1C, U3 AP2112K-3.3, U4 E73-2G4M08S1C, U5 LN2054Y42AMR, U6 AP2112K-3.3, Y1 32.768kHz, Y2 32.768kHz

Commit message: initial route done, side 1
Parts:
- removed REF** (x5): mouseBit_2.5mm, BlueSof:mouseBit_2.5mm
- removed REF**: breakaway-mousebites, Keebio-Parts:breakaway-mousebites
- added H1: MountingHole_4.5mm, MountingHole:MountingHole_4.5mm, F.Cu at (130.5, 61.4)
- added H2: MountingHole_4.5mm, MountingHole:MountingHole_4.5mm, F.Cu at (130.5, 95.4)
- added H3: MountingHole_4.5mm, MountingHole:MountingHole_4.5mm, F.Cu at (202.5, 99.7)
- added H4: MountingHole_4.5mm, MountingHole:MountingHole_4.5mm, F.Cu at (202.5, 65.7)
- added H5: MountingHole_4.5mm, MountingHole:MountingHole_4.5mm, F.Cu at (107.0, 51.0)
- added H6: MountingHole_4.5mm, MountingHole:MountingHole_4.5mm, F.Cu at (104.2, 114.4)
- added J11: SM02B-SRSS-TB(LF)(SN), BlueSof:SM02B-SRSS-TB(LF)(SN), F.Cu at (-113.5, 96.7)
- added J12: SM02B-SRSS-TB(LF)(SN), BlueSof:SM02B-SRSS-TB(LF)(SN), B.Cu at (114.7, 100.0)
- BATT1: renamed from SW59; footprint Button_Switch_THT:SW_CuK_OS102011MA1QN1_SPDT_Angled -> BlueSof:SW-TH_MSK12C02; moved to B.Cu
- C1, C2, C3, C4, C5, D1, D10, D11, D12, D13, D14, D15, D16, D17, D18, D19, D2, D20, D21, D22, D23, D24, D25, D26, D27, D28, D3, D33, D4, D5, D6, D7, D8, D9, J1, Q2, R1, R2, R4, R5, R6, R7, R8, R9, U1, U2, U3, Y1: moved to B.Cu
- RESET1: renamed from SW31; moved to B.Cu
- SW55: footprint Button_Switch_THT:SW_CuK_OS102011MA1QN1_SPDT_Angled -> BlueSof:SW-TH_MSK12C02
- SWD/C1: renamed from J3; moved to B.Cu
- USB1: renamed from J9; moved to B.Cu
- moved D32 63.3 mm to (148.6, 77.1), turned to 180 degrees
- moved R6 59.5 mm to (148.6, 78.7), turned to 180 degrees
- moved USB1 52.0 mm to (91.6, 61.1), turned to -90 degrees
- moved D31 50.8 mm to (130.4, 79.5), turned to 180 degrees
- moved R1 47.2 mm to (130.4, 81.1), turned to 180 degrees
- moved SWD/C1 35.7 mm to (99.2, 65.5), turned to 90 degrees
- moved C1 30.7 mm to (116.0, 86.1), turned to 180 degrees
- moved U1 24.1 mm to (116.0, 81.9), turned to 180 degrees
- moved R2 24.0 mm to (116.0, 84.5), turned to 0 degrees
- moved U3 19.7 mm to (107.6, 68.3), turned to 180 degrees
- moved C5 17.5 mm to (107.6, 65.9), turned to 0 degrees
- moved R9 17.3 mm to (114.2, 68.4), turned to 90 degrees
- moved Q2 16.3 mm to (111.6, 68.3)
- moved D33 15.0 mm to (111.7, 65.5), turned to 0 degrees
- moved C4 10.2 mm to (106.4, 57.9), turned to 180 degrees
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Connections:
- BATT1 pad 3: Net-(SW59-Pad3) -> no_connect_126
- D1 pad 2: col4 -> Net-(D1-Pad2)
- D16 pad 2: Net-(SW17-Pad1) -> Net-(D16-Pad2)
- D17 pad 2: Net-(SW18-Pad1) -> Net-(D17-Pad2)
- D19 pad 2: Net-(SW20-Pad1) -> Net-(D19-Pad2)
- D2 pad 2: col3 -> Net-(D2-Pad2)
- D20 pad 2: Net-(SW20-Pad2) -> Net-(D20-Pad2)
- D21 pad 2: Net-(SW22-Pad1) -> Net-(D21-Pad2)
- D22 pad 2: col1 -> Net-(D22-Pad2)
- D23 pad 2: col0 -> Net-(D23-Pad2)
- D26 pad 2: col3 -> Net-(D26-Pad2)
- D27 pad 2: col2 -> Net-(D27-Pad2)
- D3 pad 2: col2 -> Net-(D3-Pad2)
- D4 pad 2: col1 -> Net-(D4-Pad2)
- D5 pad 2: col0 -> Net-(D5-Pad2)
- D8 pad 2: Net-(SW8-Pad2) -> Net-(D8-Pad2)
- J1 pad A8: no_connect_113 -> no_connect_127
- J1 pad B8: no_connect_114 -> no_connect_128
- J7 pad A8: no_connect_115 -> no_connect_129
- J7 pad B8: no_connect_116 -> no_connect_130
- R12 pad 2: GND -> GND2
- R13 pad 2: GND -> GND2
- SW1 pad 2: col4 -> Net-(D1-Pad2)
- SW10 pad 1: Net-(D9-Pad2) -> col2
- SW11 pad 1: Net-(D10-Pad2) -> col1
- SW12 pad 1: Net-(D11-Pad2) -> col0
- SW14 pad 1: Net-(D13-Pad2) -> col4
- SW15 pad 1: Net-(D14-Pad2) -> col3
- SW16 pad 1: Net-(D15-Pad2) -> col2
- SW16 pad 2: Net-(SW17-Pad1) -> Net-(D16-Pad2)
- SW17 pad 1: Net-(SW17-Pad1) -> col1
- SW17 pad 2: Net-(SW18-Pad1) -> Net-(D17-Pad2)
- SW18 pad 1: Net-(SW18-Pad1) -> col0
- SW19 pad 2: Net-(SW20-Pad1) -> Net-(D19-Pad2)
- SW2 pad 2: col3 -> Net-(D2-Pad2)
- SW20 pad 1: Net-(SW20-Pad1) -> col4
- SW20 pad 2: Net-(SW20-Pad2) -> Net-(D20-Pad2)
- SW21 pad 1: Net-(SW20-Pad2) -> col3
- SW21 pad 2: Net-(SW22-Pad1) -> Net-(D21-Pad2)
- SW22 pad 1: Net-(SW22-Pad1) -> col2
- SW22 pad 2: col1 -> Net-(D22-Pad2)
- SW23 pad 2: col0 -> Net-(D23-Pad2)
- SW26 pad 2: col3 -> Net-(D26-Pad2)
- SW27 pad 2: col2 -> Net-(D27-Pad2)
- SW28 pad 2: Net-(SW28-Pad2) -> Net-(D28-Pad2)
- SW3 pad 2: col2 -> Net-(D3-Pad2)
- SW4 pad 2: col1 -> Net-(D4-Pad2)
- SW5 pad 2: col0 -> Net-(D5-Pad2)
- SW8 pad 1: Net-(D7-Pad2) -> col4
- SW8 pad 2: Net-(SW8-Pad2) -> Net-(D8-Pad2)
- SW9 pad 1: Net-(SW8-Pad2) -> col3
- U2 pad 12: no_connect_117 -> no_connect_131
- U2 pad 14: no_connect_118 -> no_connect_132
- U2 pad 16: no_connect_119 -> no_connect_133
- U2 pad 17: row0 -> row2
- U2 pad 18: no_connect_120 -> no_connect_134
- U2 pad 20: no_connect_121 -> no_connect_135
- U2 pad 22: no_connect_122 -> no_connect_136
- U2 pad 28: no_connect_123 -> no_connect_137
- U2 pad 30: no_connect_124 -> no_connect_138
- U2 pad 32: no_connect_125 -> no_connect_139
- U2 pad 34: no_connect_126 -> no_connect_140
- U2 pad 36: no_connect_127 -> no_connect_141
- U2 pad 38: no_connect_128 -> no_connect_142
- U2 pad 40: no_connect_129 -> no_connect_143
- U2 pad 42: no_connect_130 -> no_connect_144
- U2 pad 9: row2 -> row0
- U3 pad 4: no_connect_131 -> no_connect_145
- U4 pad 12: no_connect_132 -> no_connect_146
- U4 pad 14: no_connect_133 -> no_connect_147
- U4 pad 16: no_connect_134 -> no_connect_148
- U4 pad 18: no_connect_135 -> no_connect_149
- U4 pad 20: no_connect_136 -> no_connect_150
- U4 pad 22: no_connect_137 -> no_connect_151
- U4 pad 28: no_connect_138 -> no_connect_152
- U4 pad 30: no_connect_139 -> no_connect_153
- U4 pad 32: no_connect_140 -> no_connect_154
- U4 pad 34: no_connect_141 -> no_connect_155
- U4 pad 36: no_connect_142 -> no_connect_156
- U4 pad 38: no_connect_143 -> no_connect_157
- U4 pad 40: no_connect_144 -> no_connect_158
- U4 pad 42: no_connect_145 -> no_connect_159
- U6 pad 4: no_connect_146 -> no_connect_160
Routing:
- net col1: track 0.00 -> 205.1 mm, vias 0 -> 1
- net col0: track 0.00 -> 192.8 mm, vias 0 -> 1
- net col2: track 0.00 -> 177.8 mm, vias 0 -> 1
- net col3: track 0.00 -> 160.8 mm, vias 0 -> 1
- net row3: track 0.00 -> 158.1 mm, vias 0 -> 2
- net row2: track 0.00 -> 147.8 mm
- net col4: track 0.00 -> 139.6 mm, vias 0 -> 1
- net row0: track 0.00 -> 124.2 mm
- net row1: track 0.00 -> 121.6 mm
- net row4: track 0.00 -> 116.4 mm, vias 0 -> 2
- net VBAT: track 0.00 -> 108.1 mm, vias 0 -> 2
- net col5: track 0.00 -> 93.7 mm, vias 0 -> 1
- net VBUS: track 0.00 -> 76.7 mm, vias 0 -> 4
- net Net-(BATT1-Pad2): track 0.00 -> 74.3 mm, vias 0 -> 2
- net GND: track 0.00 -> 72.4 mm, vias 0 -> 7
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- removed copper zone on B.Cu, net GND
Other:
- board size 134.3 x 100.2 mm -> 134.8 x 98.3 mm
- board text added: "+"
- board text added: "-"
