File: PCB_RIGHT/BlueSof.kicad_sch (KiCad schematic)
At the start: 90 parts, among them J1 USB_C_Receptacle_USB2.0, J12 SM02B-SRSS-TB(LF)(SN), Q2 A03407, SW1 SW_PUSH, SW10 SW_PUSH, SW11 SW_PUSH, SW12 SW_PUSH, SW13 SW_PUSH, SW14 SW_PUSH, SW15 SW_PUSH, SW16 SW_PUSH, SW17 SW_PUSH, SW18 SW_PUSH, SW19 SW_PUSH, SW2 SW_PUSH, SW20 SW_PUSH, SW21 SW_PUSH, SW22 SW_PUSH, SW23 SW_PUSH, SW24 SW_PUSH, SW25 Rotary_Encoder_Switch, SW26 SW_PUSH, SW27 SW_PUSH, SW28 SW_PUSH, SW3 SW_PUSH, SW4 SW_PUSH, SW5 SW_PUSH, SW6 SW_PUSH, SW7 SW_PUSH, SW8 SW_PUSH, SW9 SW_PUSH, U1 LN2054Y42AMR, U2 E73-2G4M08S1C, U3 AP2112K-3.3, Y1 32.768kHz

Commit message: working towards next order
Parts:
- added BattJumper1: Jumper_2_Open, Jumper:SolderJumper-2_P1.3mm_Open_Pad1.0x1.5mm, symbol Jumper:Jumper_2_Open
- added J2, J3: Conn_01x01_Female, Connector_PinSocket_1.27mm:PinSocket_1x01_P1.27mm_Vertical, symbol Connector:Conn_01x01_Female
Connections:
- net GND: now also J3.1 (Pin_1)
- net VBAT: now also BattJumper1.1 (A)
- new net: BattJumper1.2 (B), J2.1 (Pin_1)
Changed lines of the file:
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@@
+    (stroke (width 0) (type solid) (color 0 0 0 0))
+  )
+  (wire (pts (xy 373.126 401.32) (xy 375.285 401.32))
     (stroke (width 0) (type solid) (color 0 0 0 0))
   )
@@
     (stroke (width 0) (type solid) (color 0 0 0 0))
   )
+  (wire (pts (xy 385.445 401.32) (xy 397.51 401.32))
+    (stroke (width 0) (type solid) (color 0 0 0 0))
+  )
   (wire (pts (xy 387.35 151.13) (xy 389.89 151.13))
     (stroke (width 0) (type solid) (color 0 0 0 0))
@@
   )
   (wire (pts (xy 392.43 69.85) (xy 388.62 69.85))
+    (stroke (width 0) (type solid) (color 0 0 0 0))
+  )
+  (wire (pts (xy 395.605 395.605) (xy 398.145 395.605))
     (stroke (width 0) (type solid) (color 0 0 0 0))
   )
@@
     (effects (font (size 1.27 1.27)) (justify left))
   )
+  (global_label "VBAT" (shape input) (at 373.126 401.32 180)    (property "Intersheet References" "${INTERSHEET_REFS}" (id 0) (at -120.904 222.25 0)
+      (effects (font (size 1.27 1.27)) hide)
+    )
+    (effects (font (size 1.27 1.27)) (justify right))
+  )
   (global_label "P0.05" (shape input) (at 373.38 151.13 180)    (property "Intersheet References" "${INTERSHEET_REFS}" (id 0) (at 95.25 -6.35 0)
       (effects (font (size 1.27 1.27)) hide)
@@
   )
   (global_label "VBAT" (shape input) (at 395.605 386.08 180)    (property "Intersheet References" "${INTERSHEET_REFS}" (id 0) (at -98.425 207.01 0)
+      (effects (font (size 1.27 1.27)) hide)
+    )
+    (effects (font (size 1.27 1.27)) (justify right))
+  )
+  (global_label "GND" (shape input) (at 395.605 395.605 180)    (property "Intersheet References" "${INTERSHEET_REFS}" (id 0) (at -98.425 213.995 0)
       (effects (font (size 1.27 1.27)) hide)
     )
@@
     )
   )
+  (symbol (lib_id "Connector:Conn_01x01_Female") (at 402.59 401.32 0) (unit 1)
+    (in_bom yes) (on_board yes)
+    (property "Reference" "J2" (id 0) (at 403.3013 400.6278 0)
+      (effects (font (size 1.27 1.27)) (justify left))
+    )
+    (property "Value" "Conn_01x01_Female" (id 1) (at 407.1113 401.0215 0)
+      (effects (font (size 1.27 1.27)) (justify left))
+    )
+    (property "Footprint" "Connector_PinSocket_1.27mm:PinSocket_1x01_P1.27mm_Vertical" (id 2) (at 402.59 401.32 0)
+      (effects (font (size 1.27 1.27)) hide)
+    )
+    (property "Datasheet" "~" (id 3) (at 402.59 401.32 0)
+      (effects (font (size 1.27 1.27)) hide)
+    )
+  )
+  (symbol (lib_id "Connector:Conn_01x01_Female") (at 403.225 395.605 0) (unit 1)
+    (in_bom yes) (on_board yes)
+    (property "Reference" "J3" (id 0) (at 403.9363 394.9128 0)
+      (effects (font (size 1.27 1.27)) (justify left))
+    )
+    (property "Value" "Conn_01x01_Female" (id 1) (at 407.7463 395.3065 0)
+      (effects (font (size 1.27 1.27)) (justify left))
+    )
+    (property "Footprint" "Connector_PinSocket_1.27mm:PinSocket_1x01_P1.27mm_Vertical" (id 2) (at 403.225 395.605 0)
+      (effects (font (size 1.27 1.27)) hide)
+    )
+    (property "Datasheet" "~" (id 3) (at 403.225 395.605 0)
+      (effects (font (size 1.27 1.27)) hide)
+    )
+  )
   (symbol (lib_id "Device:C_Small") (at 349.25 140.97 0) (unit 1)
     (in_bom yes) (on_board yes)
@@
     )
   )
+  (symbol (lib_id "Jumper:Jumper_2_Open") (at 380.365 401.32 0) (unit 1)
+    (in_bom yes) (on_board yes)
+    (property "Reference" "BattJumper1" (id 0) (at 380.365 395.459 0))
+    (property "Value" "Jumper_2_Open" (id 1) (at 380.365 397.7575 0))
+    (property "Footprint" "Jumper:SolderJumper-2_P1.3mm_Open_Pad1.0x1.5mm" (id 2) (at 380.365 401.32 0)
+      (effects (font (size 1.27 1.27)) hide)
+    )
+    (property "Datasheet" "~" (id 3) (at 380.365 401.32 0)
+      (effects (font (size 1.27 1.27)) hide)
+    )
+  )
   (symbol (lib_id "Switch:SW_Push") (at 335.28 257.81 0) (unit 1)
     (in_bom yes) (on_board yes)
@@
       (reference "BATT1") (unit 1) (value "SW_SPDT") (footprint "BlueSof:SW-TH_MSK12C02")
     )
+    (path "/93bd7854-a686-46a4-8788-974af210b24a"
+      (reference "BattJumper1") (unit 1) (value "Jumper_2_Open") (footprint "Jumper:SolderJumper-2_P1.3mm_Open_Pad1.0x1.5mm")
+    )
     (path "/00000000-0000-0000-0000-00005fd31558"
       (reference "C1") (unit 1) (value "4.7uF") (footprint "Capacitor_SMD:C_0603_1608Metric")
@@
       (reference "J1") (unit 1) (value "USB_C_Receptacle_USB2.0") (footprint "BlueSof:USB-C_C168688")
     )
+    (path "/f7654d63-c254-4fa6-9277-48d1c993b521"
+      (reference "J2") (unit 1) (value "Conn_01x01_Female") (footprint "Connector_PinSocket_1.27mm:PinSocket_1x01_P1.27mm_Vertical")
+    )
+    (path "/5854e4fc-3f3d-4fb1-946a-a29dc023b373"
+      (reference "J3") (unit 1) (value "Conn_01x01_Female") (footprint "Connector_PinSocket_1.27mm:PinSocket_1x01_P1.27mm_Vertical")
+    )
     (path "/854d8cf3-8c16-4b20-a5e1-a1229cd64724"
