File: PCB/SP56/SP56.kicad_pcb (KiCad board)
At the start: 2 copper layers, 272.1 x 98.3 mm, 193 parts, among them J1 USB_C_Receptacle_USB2.0, J101 USB_C_Receptacle_USB2.0, J103 Conn_01x01_Female, J104 Conn_01x01_Female, J106 SM02B-SRSS-TB(LF)(SN), J2 Conn_01x01_Male, J3 Conn_01x01_Male, J9 SM02B-SRSS-TB(LF)(SN), Q1 A03407, Q102 A03407, SW1 SW_PUSH, SW10 SW_PUSH, SW101 SW_PUSH, SW102 SW_PUSH, SW103 SW_PUSH, SW104 SW_PUSH, SW105 SW_PUSH, SW106 SW_PUSH, SW107 SW_PUSH, SW108 SW_PUSH, SW109 SW_PUSH, SW11 SW_PUSH, SW110 SW_PUSH, SW111 SW_PUSH, SW112 SW_PUSH, SW113 SW_PUSH, SW114 SW_PUSH, SW115 SW_PUSH, SW116 SW_PUSH, SW117 SW_PUSH, SW118 SW_PUSH, SW119 SW_PUSH, SW12 SW_PUSH, SW120 SW_PUSH, SW121 SW_PUSH, SW122 SW_PUSH, SW123 SW_PUSH, SW124 SW_PUSH, SW125 Rotary_Encoder_Switch, SW126 SW_PUSH, SW127 SW_PUSH, SW128 SW_PUSH, SW13 SW_PUSH, SW14 SW_PUSH, SW15 SW_PUSH, SW16 SW_PUSH, SW17 SW_PUSH, SW18 SW_PUSH, SW19 SW_PUSH, SW2 SW_PUSH, SW20 SW_PUSH, SW21 SW_PUSH, SW22 SW_PUSH, SW23 SW_PUSH, SW24 SW_PUSH, SW25 Rotary_Encoder_Switch, SW26 SW_PUSH, SW27 SW_PUSH, SW28 SW_PUSH, SW3 SW_PUSH, SW4 SW_PUSH, SW5 SW_PUSH, SW6 SW_PUSH, SW7 SW_PUSH, SW8 SW_PUSH, SW9 SW_PUSH, U1 LN2054Y42AMR, U101 LN2054Y42AMR, U102 E73-2G4M08S1C, U103 AP2112K-3.3, U2 E73-2G4M08S1C, U3 AP2112K-3.3, Y1 32.768kHz, Y101 32.768kHz

Commit message: ready for jlc quote
Parts:
- U102, U2: footprint BlueSof:E73-2G4M08S1C-52840_SMD -> BlueSof:E73-2G4M08S1C_LCSC
- moved C1 7.17 mm to (341.0, 29.4), turned to 90 degrees
- moved U102 7.10 mm to (114.9, 17.5), turned to 0 degrees
- moved U2 7.00 mm to (334.1, 17.6), turned to 0 degrees
- moved C2 2.92 mm to (342.5, 29.4)
- moved Y1 2.54 mm to (340.4, 26.8)
- moved Y101 0.84 mm to (118.7, 26.7)
- moved D1 0.80 mm to (324.4, 8.65)
- moved R1 0.62 mm to (343.3, 11.7)
- moved C103 0.40 mm to (122.3, 27.0)
- moved C104 0.40 mm to (122.3, 25.4)
- moved J9 0.38 mm to (336.8, 29.2)
Routing:
- net /SP56_Left/BATTERY_MEASURE: track 34.3 -> 55.3 mm
- net /SP56_Left/VBUS: track 80.0 -> 94.3 mm, vias 4 -> 6
- net /SP56_Right/col0: track 157.8 -> 144.9 mm
- net GND: track 75.0 -> 86.5 mm, vias 112 -> 113
- net /SP56_Right/VDD_H: track 23.3 -> 14.0 mm, vias 1 -> 0
- net /SP56_Left/VDD_H: track 32.9 -> 24.1 mm, vias 0 -> 2
- net /SP56_Left/row1: track 137.7 -> 128.9 mm
- net /SP56_Left/RESET: track 39.1 -> 44.1 mm
- net /SP56_Left/SWD: track 5.94 -> 8.99 mm
- net /SP56_Left/col3: track 153.5 -> 150.5 mm
- net Net-(C1-Pad2): track 3.35 -> 6.23 mm
- net /SP56_Right/SWD: track 5.30 -> 7.53 mm
- net Net-(C2-Pad2): track 4.07 -> 6.24 mm
- net Net-(D1-Pad2): track 24.2 -> 22.0 mm
- net Net-(C103-Pad2): track 5.27 -> 7.00 mm
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
Commit message: order SP56 R1 from JLC
Parts:
- removed BattJumper1, BattJumper101: Jumper_2_Open, Jumper:SolderJumper-2_P1.3mm_Open_Pad1.0x1.5mm
- added C8: 4.7nF, Capacitor_SMD:C_0603_1608Metric, B.Cu at (342.8, 6.40)
- added C9: 4.7nF, Capacitor_SMD:C_0603_1608Metric, B.Cu at (106.1, 8.20)
- added R10: 1M, Resistor_SMD:R_0603_1608Metric, B.Cu at (106.1, 6.70)
- added R3: 1M, Resistor_SMD:R_0603_1608Metric, B.Cu at (342.8, 8.00)
Connections:
- J1 pad S1: unconnected-(J1-PadS1) -> Net-(C8-Pad1)
- J101 pad S1: unconnected-(J101-PadS1) -> Net-(C9-Pad1)
- J104 pad 1: Net-(BattJumper101-Pad2) -> /SP56_Right/VBAT
- J3 pad 1: Net-(BattJumper1-Pad2) -> /SP56_Left/VBAT
Routing:
- net /SP56_Right/VBAT: track 51.4 -> 68.9 mm
- net Net-(BattJumper1-Pad2): track 17.1 -> 0.00 mm
- net /SP56_Left/VBAT: track 46.3 -> 61.9 mm
- net Net-(BattJumper101-Pad2): track 14.9 -> 0.00 mm
- net Net-(C9-Pad1): track 0.00 -> 13.6 mm
- net Net-(C8-Pad1): track 0.00 -> 13.5 mm
- net GND: track 86.5 -> 99.3 mm, vias 113 -> 119
- net unconnected-(J101-PadS1): track 10.0 -> 0.00 mm
- net unconnected-(J1-PadS1): track 10.0 -> 0.00 mm
- net Net-(D31-Pad1): track 5.75 -> 2.53 mm
- net /SP56_Left/col4: track 141.4 -> 142.9 mm
- net /SP56_Left/col3: track 150.5 -> 151.6 mm
- net /SP56_Left/col5: track 99.2 -> 99.9 mm
Other:
- board text added: "OFF ON"
- board text added: "ON OFF"
