File: PCB/SP56/SP56_Left.kicad_sch (KiCad schematic)
At the start: 95 parts, among them J1 USB_C_Receptacle_USB2.0, J2 Conn_01x01_Male, J3 Conn_01x01_Male, J9 SM02B-SRSS-TB(LF)(SN), Q1 A03407, SW1 SW_PUSH, SW10 SW_PUSH, SW11 SW_PUSH, SW12 SW_PUSH, SW13 SW_PUSH, SW14 SW_PUSH, SW15 SW_PUSH, SW16 SW_PUSH, SW17 SW_PUSH, SW18 SW_PUSH, SW19 SW_PUSH, SW2 SW_PUSH, SW20 SW_PUSH, SW21 SW_PUSH, SW22 SW_PUSH, SW23 SW_PUSH, SW24 SW_PUSH, SW25 Rotary_Encoder_Switch, SW26 SW_PUSH, SW27 SW_PUSH, SW28 SW_PUSH, SW3 SW_PUSH, SW4 SW_PUSH, SW5 SW_PUSH, SW6 SW_PUSH, SW7 SW_PUSH, SW8 SW_PUSH, SW9 SW_PUSH, U1 LN2054Y42AMR, U2 E73-2G4M08S1C, U3 AP2112K-3.3, Y1 32.768kHz

Commit message: ready for jlc quote
Other:
- note added: "LED"
- company: (none) -> CO Boards
- title: (none) -> SP56
- moved on the sheet: BATT1, BattJumper1, C1, C2, C3, C4, C5, C6, C7, D1, D10, D11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

Commit message: order SP56 R1 from JLC
Parts:
- removed BattJumper1: Jumper_2_Open, Jumper:SolderJumper-2_P1.3mm_Open_Pad1.0x1.5mm, symbol Jumper:Jumper_2_Open
- added C8: 4.7nF, Capacitor_SMD:C_0603_1608Metric, symbol Device:C_Small
- added R3: 1M, Resistor_SMD:R_0603_1608Metric, symbol Device:R_Small
Connections:
- net GND: now also C8.2, R3.2
- net VBAT: now also J3.1 (Pin_1)
- net at J1.S1 (SHIELD): now also C8.1, R3.1
- no-connect marks 26 -> 25
Changed lines of the file:
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@@
   (junction (at 110.49 151.13) (diameter 1.016) (color 0 0 0 0))
   (junction (at 110.49 167.64) (diameter 1.016) (color 0 0 0 0))
+  (junction (at 120.65 64.77) (diameter 1.016) (color 0 0 0 0))
+  (junction (at 123.19 72.39) (diameter 1.016) (color 0 0 0 0))
+  (junction (at 125.73 72.39) (diameter 1.016) (color 0 0 0 0))
   (junction (at 125.73 125.73) (diameter 1.016) (color 0 0 0 0))
   (junction (at 125.73 142.24) (diameter 1.016) (color 0 0 0 0))
@@
   (no_connect (at 60.96 36.83))
   (no_connect (at 66.04 36.83))
-  (no_connect (at 120.65 64.77))
   (no_connect (at 143.51 54.61))
   (no_connect (at 143.51 57.15))
@@
     (stroke (width 0) (type solid) (color 0 0 0 0))
   )
+  (wire (pts (xy 118.11 64.77) (xy 120.65 64.77))
+    (stroke (width 0) (type solid) (color 0 0 0 0))
+  )
+  (wire (pts (xy 118.11 66.04) (xy 118.11 64.77))
+    (stroke (width 0) (type solid) (color 0 0 0 0))
+  )
+  (wire (pts (xy 118.11 71.12) (xy 118.11 72.39))
+    (stroke (width 0) (type solid) (color 0 0 0 0))
+  )
+  (wire (pts (xy 118.11 72.39) (xy 123.19 72.39))
+    (stroke (width 0) (type solid) (color 0 0 0 0))
+  )
+  (wire (pts (xy 123.19 64.77) (xy 120.65 64.77))
+    (stroke (width 0) (type solid) (color 0 0 0 0))
+  )
+  (wire (pts (xy 123.19 66.04) (xy 123.19 64.77))
+    (stroke (width 0) (type solid) (color 0 0 0 0))
+  )
+  (wire (pts (xy 123.19 71.12) (xy 123.19 72.39))
+    (stroke (width 0) (type solid) (color 0 0 0 0))
+  )
+  (wire (pts (xy 123.19 72.39) (xy 125.73 72.39))
+    (stroke (width 0) (type solid) (color 0 0 0 0))
+  )
   (wire (pts (xy 123.19 118.11) (xy 125.73 118.11))
     (stroke (width 0) (type solid) (color 0 0 0 0))
@@
     (stroke (width 0) (type solid) (color 0 0 0 0))
   )
-  (wire (pts (xy 124.46 67.31) (xy 128.27 67.31))
+  (wire (pts (xy 125.73 72.39) (xy 128.27 72.39))
     (stroke (width 0) (type solid) (color 0 0 0 0))
   )
@@
     (stroke (width 0) (type solid) (color 0 0 0 0))
   )
+  (wire (pts (xy 128.27 67.31) (xy 128.27 72.39))
+    (stroke (width 0) (type solid) (color 0 0 0 0))
+  )
   (wire (pts (xy 130.81 118.11) (xy 130.81 134.62))
     (stroke (width 0) (type solid) (color 0 0 0 0))
@@
     (stroke (width 0) (type solid) (color 0 0 0 0))
   )
-  (wire (pts (xy 242.824 154.94) (xy 242.824 161.29))
-    (stroke (width 0) (type solid) (color 0 0 0 0))
-  )
-  (wire (pts (xy 242.824 154.94) (xy 246.38 154.94))
-    (stroke (width 0) (type solid) (color 0 0 0 0))
-  )
-  (wire (pts (xy 242.824 161.29) (xy 235.839 161.29))
-    (stroke (width 0) (type solid) (color 0 0 0 0))
-  )
   (wire (pts (xy 243.84 121.92) (xy 245.11 121.92))
     (stroke (width 0) (type solid) (color 0 0 0 0))
@@
   )
   (wire (pts (xy 243.84 151.13) (xy 246.38 151.13))
+    (stroke (width 0) (type solid) (color 0 0 0 0))
+  )
+  (wire (pts (xy 243.84 154.94) (xy 246.38 154.94))
     (stroke (width 0) (type solid) (color 0 0 0 0))
   )
@@
     (effects (font (size 1.27 1.27)) (justify right bottom))
   )
-  (label "VBAT" (at 225.679 161.29 180)
-    (effects (font (size 1.27 1.27)) (justify right bottom))
-  )
   (label "BATT_SWITCHED" (at 236.22 29.21 180)
     (effects (font (size 1.27 1.27)) (justify right bottom))
@@
   )
   (label "GND" (at 243.84 151.13 180)
+    (effects (font (size 1.27 1.27)) (justify right bottom))
+  )
+  (label "VBAT" (at 243.84 154.94 180)
     (effects (font (size 1.27 1.27)) (justify right bottom))
   )
@@
     )
   )
-  (symbol (lib_id "power:GND") (at 124.46 67.31 0) (unit 1)
-    (in_bom yes) (on_board yes)
-    (property "Reference" "#PWR05" (id 0) (at 124.46 73.66 0)
-      (effects (font (size 1.27 1.27)) hide)
-    )
-    (property "Value" "GND" (id 1) (at 124.587 71.7042 0))
-    (property "Footprint" "" (id 2) (at 124.46 67.31 0)
-      (effects (font (size 1.27 1.27)) hide)
-    )
-    (property "Datasheet" "" (id 3) (at 124.46 67.31 0)
+  (symbol (lib_id "power:GND") (at 125.73 72.39 0) (unit 1)
+    (in_bom yes) (on_board yes)
+    (property "Reference" "#PWR05" (id 0) (at 125.73 78.74 0)
+      (effects (font (size 1.27 1.27)) hide)
+    )
+    (property "Value" "GND" (id 1) (at 125.857 76.7842 0))
+    (property "Footprint" "" (id 2) (at 125.73 72.39 0)
+      (effects (font (size 1.27 1.27)) hide)
+    )
+    (property "Datasheet" "" (id 3) (at 125.73 72.39 0)
       (effects (font (size 1.27 1.27)) hide)
     )
@@
     )
     (property "Datasheet" "" (id 3) (at 275.59 127 0)
+      (effects (font (size 1.27 1.27)) hide)
+    )
+  )
+  (symbol (lib_id "Device:R_Small") (at 118.11 68.58 0) (unit 1)
+    (in_bom yes) (on_board yes)
+    (property "Reference" "R3" (id 0) (at 114.5287 71.2406 0)
+      (effects (font (size 1.27 1.27)) (justify left))
+    )
+    (property "Value" "1M" (id 1) (at 115.799 67.189 90)
+      (effects (font (size 1.27 1.27)) (justify left))
+    )
+    (property "Footprint" "Resistor_SMD:R_0603_1608Metric" (id 2) (at 118.11 68.58 0)
+      (effects (font (size 1.27 1.27)) hide)
+    )
+    (property "Datasheet" "~" (id 3) (at 118.11 68.58 0)
       (effects (font (size 1.27 1.27)) hide)
     )
@@
     )
   )
+  (symbol (lib_id "Device:C_Small") (at 123.19 68.58 0) (unit 1)
+    (in_bom yes) (on_board yes)
+    (property "Reference" "C8" (id 0) (at 120.4342 71.2406 0)
+      (effects (font (size 1.27 1.27)) (justify left))
+    )
+    (property "Value" "4.7nF" (id 1) (at 124.244 67.189 90)
+      (effects (font (size 1.27 1.27)) (justify left))
+    )
+    (property "Footprint" "Capacitor_SMD:C_0603_1608Metric" (id 2) (at 123.19 68.58 0)
+      (effects (font (size 1.27 1.27)) hide)
+    )
+    (property "Datasheet" "~" (id 3) (at 123.19 68.58 0)
+      (effects (font (size 1.27 1.27)) hide)
+    )
+  )
   (symbol (lib_id "Device:C_Small") (at 179.07 50.8 0) (unit 1)
     (in_bom yes) (on_board yes)
@@
       (effects (font (size 1.27 1.27)) hide)
     )
-  )
-  (symbol (lib_id "Jumper:Jumper_2_Open") (at 230.759 161.29 0) (unit 1)
-    (in_bom yes) (on_board yes)
-    (property "Reference" "BattJumper1" (id 0) (at 230.759 155.429 0))
-    (property "Value" "Jumper_2_Open" (id 1) (at 230.759 157.7275 0))
-    (property "Footprint" "Jumper:SolderJumper-2_P1.3mm_Open_Pad1.0x1.5mm" (id 2) (at 230.759 161.29 0)
-      (effects (font (size 1.27 1.27)) hide)
-    )
-    (property "Datasheet" "~" (id 3) (at 230.759 161.29 0)
-      (effects (font (size 1.27 1.27)) hide)
-    )
