File: PCB/SP56/SP56_Right.kicad_sch (KiCad schematic)
At the start: 95 parts, among them J101 USB_C_Receptacle_USB2.0, J103 Conn_01x01_Female, J104 Conn_01x01_Female, J106 SM02B-SRSS-TB(LF)(SN), Q102 A03407, SW101 SW_PUSH, SW102 SW_PUSH, SW103 SW_PUSH, SW104 SW_PUSH, SW105 SW_PUSH, SW106 SW_PUSH, SW107 SW_PUSH, SW108 SW_PUSH, SW109 SW_PUSH, SW110 SW_PUSH, SW111 SW_PUSH, SW112 SW_PUSH, SW113 SW_PUSH, SW114 SW_PUSH, SW115 SW_PUSH, SW116 SW_PUSH, SW117 SW_PUSH, SW118 SW_PUSH, SW119 SW_PUSH, SW120 SW_PUSH, SW121 SW_PUSH, SW122 SW_PUSH, SW123 SW_PUSH, SW124 SW_PUSH, SW125 Rotary_Encoder_Switch, SW126 SW_PUSH, SW127 SW_PUSH, SW128 SW_PUSH, U101 LN2054Y42AMR, U102 E73-2G4M08S1C, U103 AP2112K-3.3, Y101 32.768kHz

Commit message: ready for jlc quote
Other:
- note added: "LED"
- company: (none) -> CO Boards
- title: (none) -> SP56
- moved on the sheet: BATT101, BattJumper101, C101, C102, C103, C104, C105, C106, C107, D101, D102, D103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

Commit message: order SP56 R1 from JLC
Parts:
- removed BattJumper101: Jumper_2_Open, Jumper:SolderJumper-2_P1.3mm_Open_Pad1.0x1.5mm, symbol Jumper:Jumper_2_Open
- added C9: 4.7nF, Capacitor_SMD:C_0603_1608Metric, symbol Device:C_Small
- added R10: 1M, Resistor_SMD:R_0603_1608Metric, symbol Device:R_Small
Connections:
- net GND: now also C9.2, R10.2
- net VBAT: now also J104.1 (Pin_1)
- net at J101.S1 (SHIELD): now also C9.1, R10.1
- no-connect marks 26 -> 25
Other:
- moved on the sheet: J104
Changed lines of the file:
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@@
   (junction (at 113.03 154.94) (diameter 1.016) (color 0 0 0 0))
   (junction (at 113.03 171.45) (diameter 1.016) (color 0 0 0 0))
+  (junction (at 116.84 66.04) (diameter 1.016) (color 0 0 0 0))
+  (junction (at 119.38 73.66) (diameter 1.016) (color 0 0 0 0))
+  (junction (at 124.46 73.66) (diameter 1.016) (color 0 0 0 0))
   (junction (at 128.27 129.54) (diameter 1.016) (color 0 0 0 0))
   (junction (at 128.27 146.05) (diameter 1.016) (color 0 0 0 0))
@@
   (no_connect (at 64.77 36.83))
   (no_connect (at 69.85 36.83))
-  (no_connect (at 116.84 66.04))
   (no_connect (at 139.7 55.88))
   (no_connect (at 139.7 58.42))
@@
     (stroke (width 0) (type solid) (color 0 0 0 0))
   )
-  (wire (pts (xy 120.65 68.58) (xy 124.46 68.58))
-    (stroke (width 0) (type solid) (color 0 0 0 0))
-  )
-  (wire (pts (xy 124.46 68.58) (xy 124.46 66.04))
+  (wire (pts (xy 114.3 66.04) (xy 116.84 66.04))
+    (stroke (width 0) (type solid) (color 0 0 0 0))
+  )
+  (wire (pts (xy 114.3 67.31) (xy 114.3 66.04))
+    (stroke (width 0) (type solid) (color 0 0 0 0))
+  )
+  (wire (pts (xy 114.3 72.39) (xy 114.3 73.66))
+    (stroke (width 0) (type solid) (color 0 0 0 0))
+  )
+  (wire (pts (xy 114.3 73.66) (xy 119.38 73.66))
+    (stroke (width 0) (type solid) (color 0 0 0 0))
+  )
+  (wire (pts (xy 119.38 66.04) (xy 116.84 66.04))
+    (stroke (width 0) (type solid) (color 0 0 0 0))
+  )
+  (wire (pts (xy 119.38 67.31) (xy 119.38 66.04))
+    (stroke (width 0) (type solid) (color 0 0 0 0))
+  )
+  (wire (pts (xy 119.38 72.39) (xy 119.38 73.66))
+    (stroke (width 0) (type solid) (color 0 0 0 0))
+  )
+  (wire (pts (xy 119.38 73.66) (xy 124.46 73.66))
+    (stroke (width 0) (type solid) (color 0 0 0 0))
+  )
+  (wire (pts (xy 124.46 66.04) (xy 124.46 73.66))
     (stroke (width 0) (type solid) (color 0 0 0 0))
   )
@@
     (stroke (width 0) (type solid) (color 0 0 0 0))
   )
-  (wire (pts (xy 226.441 163.195) (xy 228.6 163.195))
-    (stroke (width 0) (type solid) (color 0 0 0 0))
-  )
   (wire (pts (xy 229.87 45.72) (xy 234.95 45.72))
     (stroke (width 0) (type solid) (color 0 0 0 0))
@@
     (stroke (width 0) (type solid) (color 0 0 0 0))
   )
-  (wire (pts (xy 238.76 163.195) (xy 250.825 163.195))
-    (stroke (width 0) (type solid) (color 0 0 0 0))
-  )
   (wire (pts (xy 242.57 128.27) (xy 243.84 128.27))
     (stroke (width 0) (type solid) (color 0 0 0 0))
@@
   )
   (wire (pts (xy 248.92 160.02) (xy 251.46 160.02))
+    (stroke (width 0) (type solid) (color 0 0 0 0))
+  )
+  (wire (pts (xy 248.92 163.195) (xy 251.46 163.195))
     (stroke (width 0) (type solid) (color 0 0 0 0))
   )
@@
     (effects (font (size 1.27 1.27)) (justify right bottom))
   )
-  (label "VBAT" (at 226.441 163.195 180)
-    (effects (font (size 1.27 1.27)) (justify right bottom))
-  )
   (label "P0.05" (at 234.95 128.27 180)
     (effects (font (size 1.27 1.27)) (justify right bottom))
@@
   )
   (label "GND" (at 248.92 160.02 180)
+    (effects (font (size 1.27 1.27)) (justify right bottom))
+  )
+  (label "VBAT" (at 248.92 163.195 180)
     (effects (font (size 1.27 1.27)) (justify right bottom))
   )
@@
     )
   )
-  (symbol (lib_id "power:GND") (at 120.65 68.58 0) (unit 1)
-    (in_bom yes) (on_board yes)
-    (property "Reference" "#PWR020" (id 0) (at 120.65 74.93 0)
-      (effects (font (size 1.27 1.27)) hide)
-    )
-    (property "Value" "GND" (id 1) (at 120.777 72.9742 0))
-    (property "Footprint" "" (id 2) (at 120.65 68.58 0)
-      (effects (font (size 1.27 1.27)) hide)
-    )
-    (property "Datasheet" "" (id 3) (at 120.65 68.58 0)
+  (symbol (lib_id "power:GND") (at 124.46 73.66 0) (unit 1)
+    (in_bom yes) (on_board yes)
+    (property "Reference" "#PWR020" (id 0) (at 124.46 80.01 0)
+      (effects (font (size 1.27 1.27)) hide)
+    )
+    (property "Value" "GND" (id 1) (at 124.587 78.0542 0))
+    (property "Footprint" "" (id 2) (at 124.46 73.66 0)
+      (effects (font (size 1.27 1.27)) hide)
+    )
+    (property "Datasheet" "" (id 3) (at 124.46 73.66 0)
       (effects (font (size 1.27 1.27)) hide)
     )
@@
     )
     (property "Datasheet" "" (id 3) (at 276.86 132.08 0)
+      (effects (font (size 1.27 1.27)) hide)
+    )
+  )
+  (symbol (lib_id "Device:R_Small") (at 114.3 69.85 0) (unit 1)
+    (in_bom yes) (on_board yes)
+    (property "Reference" "R10" (id 0) (at 110.7187 72.5106 0)
+      (effects (font (size 1.27 1.27)) (justify left))
+    )
+    (property "Value" "1M" (id 1) (at 111.989 68.459 90)
+      (effects (font (size 1.27 1.27)) (justify left))
+    )
+    (property "Footprint" "Resistor_SMD:R_0603_1608Metric" (id 2) (at 114.3 69.85 0)
+      (effects (font (size 1.27 1.27)) hide)
+    )
+    (property "Datasheet" "~" (id 3) (at 114.3 69.85 0)
       (effects (font (size 1.27 1.27)) hide)
     )
@@
     )
   )
-  (symbol (lib_id "Connector:Conn_01x01_Female") (at 255.905 163.195 0) (unit 1)
-    (in_bom yes) (on_board yes)
-    (property "Reference" "J104" (id 0) (at 256.6163 162.5028 0)
-      (effects (font (size 1.27 1.27)) (justify left))
-    )
-    (property "Value" "Conn_01x01_Female" (id 1) (at 260.4263 162.8965 0)
-      (effects (font (size 1.27 1.27)) (justify left))
-    )
-    (property "Footprint" "Connector_PinSocket_1.27mm:PinSocket_1x01_P1.27mm_Vertical" (id 2) (at 255.905 163.195 0)
-      (effects (font (size 1.27 1.27)) hide)
-    )
-    (property "Datasheet" "~" (id 3) (at 255.905 163.195 0)
-      (effects (font (size 1.27 1.27)) hide)
-    )
-  )
   (symbol (lib_id "Connector:Conn_01x01_Female") (at 256.54 160.02 0) (unit 1)
     (in_bom yes) (on_board yes)
@@
     )
   )
+  (symbol (lib_id "Connector:Conn_01x01_Female") (at 256.54 163.195 0) (unit 1)
+    (in_bom yes) (on_board yes)
+    (property "Reference" "J104" (id 0) (at 257.2513 162.5028 0)
+      (effects (font (size 1.27 1.27)) (justify left))
+    )
+    (property "Value" "Conn_01x01_Female" (id 1) (at 261.0613 162.8965 0)
+      (effects (font (size 1.27 1.27)) (justify left))
+    )
+    (property "Footprint" "Connector_PinSocket_1.27mm:PinSocket_1x01_P1.27mm_Vertical" (id 2) (at 256.54 163.195 0)
+      (effects (font (size 1.27 1.27)) hide)
+    )
+    (property "Datasheet" "~" (id 3) (at 256.54 163.195 0)
+      (effects (font (size 1.27 1.27)) hide)
+    )
+  )
   (symbol (lib_id "Device:C_Small") (at 34.29 182.88 0) (unit 1)
     (in_bom yes) (on_board yes)
@@
     )
     (property "PRICE" "100k" (id 5) (at 73.66 17.78 0)
+      (effects (font (size 1.27 1.27)) hide)
+    )
+  )
+  (symbol (lib_id "Device:C_Small") (at 119.38 69.85 0) (unit 1)
+    (in_bom yes) (on_board yes)
+    (property "Reference" "C9" (id 0) (at 116.6242 72.5106 0)
+      (effects (font (size 1.27 1.27)) (justify left))
+    )
+    (property "Value" "4.7nF" (id 1) (at 120.434 68.459 90)
+      (effects (font (size 1.27 1.27)) (justify left))
+    )
+    (property "Footprint" "Capacitor_SMD:C_0603_1608Metric" (id 2) (at 119.38 69.85 0)
+      (effects (font (size 1.27 1.27)) hide)
+    )
+    (property "Datasheet" "~" (id 3) (at 119.38 69.85 0)
       (effects (font (size 1.27 1.27)) hide)
     )
@@
       (effects (font (size 1.27 1.27)) hide)
     )
-  )
-  (symbol (lib_id "Jumper:Jumper_2_Open") (at 233.68 163.195 0) (unit 1)
-    (in_bom yes) (on_board yes)
-    (property "Reference" "BattJumper101" (id 0) (at 233.68 157.334 0))
-    (property "Value" "Jumper_2_Open" (id 1) (at 233.68 159.6325 0))
-    (property "Footprint" "Jumper:SolderJumper-2_P1.3mm_Open_Pad1.0x1.5mm" (id 2) (at 233.68 163.195 0)
-      (effects (font (size 1.27 1.27)) hide)
-    )
-    (property "Datasheet" "~" (id 3) (at 233.68 163.195 0)
-      (effects (font (size 1.27 1.27)) hide)
-    )
